Commit message: Updated lidar link inertia

File: mini_pupper_2_description/urdf/mini_pupper_description.urdf.xacro (robot description, xacro)
@@ -364,15 +364,18 @@
     name="lidar_link">
     <inertial>
+      <!-- from meshlab -->
       <origin
-        xyz="1.56706411611127E-05 -5.16565672073303E-13 -0.0191835739440227"
+        xyz="0.000024 -0.001577 -0.019199"
         rpy="0 0 -1.57" />
-      <mass value="0.0001" />
+      <!-- from datasheet -->
+      <mass value="0.042" />
+      <!-- from meshlab -->
       <inertia
-        ixx="8.74731426973985E-06"
-        ixy="-6.66781590704156E-08"
-        ixz="1.89196685410159E-11"
-        iyy="8.70097486591694E-06"
-        iyz="-1.13397577799603E-17"
-        izz="9.98821295317784E-06" />
+        ixx="92.990494e-7"
+        ixy="0.6376200e-7"
+        ixz="-0.001543e-7"
+        iyy="93.455414e-7"
+        iyz="-0.101909e-7"
+        izz="99.498268e-7" />
     </inertial>
     <visual>
